File: rev_a/mini_bridge_encoders_sonar.sch (KiCad schematic (older format))
At the start: 4 parts

Commit message: Initial schematic complete.
Parts:
- added C1, C3: 22uF, symbol C_VERT
- added C2, C4: .1uF, symbol C_VERT
- added J1: POWER_SELECT, symbol POWER_SELECT
- added N10, N9: MOTOR_CONNECTOR, symbol MOTOR_CONNECTOR
- added N3, N4: ENCODER_CONNECTOR, symbol ENCODER_CONNECTOR
- added N5, N6, N7, N8: HC_SR04_CONNECTOR, symbol HC_SR04_CONNECTOR
- added R1: .47, symbol R_HORIZ
- added R10, R11, R12, R13, R8, R9: 10K, symbol R_VERT
- added R2, R3, R4, R5, R6, R7: 470, symbol R_HORIZ
- added U1: LM2940, symbol VOLTAGE_REGULATOR
- added U2, U3, U4: OPTO_ISOLATOR, symbol OPTO_ISOLATOR
- added U5: 754410, symbol 754410
Connections:
- net 5V: now also N3.4 (5V), N4.4 (5V), N5.4 (5V), N6.4 (5V), N7.4 (5V), N8.4 (5V)
- net A0: now also N8.2 (ECHO)
- net A1: now also N7.2 (ECHO)
- net A2: now also N6.2 (ECHO)
- net A3: now also N5.2 (ECHO)
- net D0: now also N8.3 (TRIG)
- net D1: now also N7.3 (TRIG)
- net D10: now also R6.1
- net D11: now also R3.1
- net D12: now also R4.1
- net D13: now also R2.1
- net D2: now also N4.2 (A)
- net D3: now also N6.3 (TRIG)
- net D4: now also N4.3 (B)
- net D5: now also N3.2 (A)
- net D6: now also N3.3 (B)
- net D7: now also R7.1
- net D8: now also R5.1
- net D9: now also N5.3 (TRIG)
- net GND: now also N3.1 (GND), N4.1 (GND), N5.1 (GND), N6.1 (GND), N7.1 (GND), N8.1 (GND), U2.2, U2.4, U3.2, U3.4, U4.2, U4.4
- net MGND: now also C1.2, C3.2, C4.1, C4.2, R1.1, R10.1, R11.1, R12.1, R13.1, R8.1, R9.1, U1.2, U5.12 (GND), U5.13 (GND), U5.4 (GND), U5.5 (GND)
- net MPWR: now also C1.1, J1.1 (VIN1), U1.1 (VIN)
- new net: R3.2, U2.3
- new net: R9.2, U2.5, U5.1 (EN12)
- new net: C2.2, R1.2
- new net: R5.2, U3.3
- new net: R11.2, U3.5, U5.10 (3A)
- new net: R6.2, U4.1
- new net: R12.2, U4.7, U5.9 (EN34)
- new net: R7.2, U4.3
- new net: R13.2, U4.5, U5.15 (4A)
- new net: R2.2, U2.1
- new net: R8.2, U2.7, U5.2 (1A)
- new net: R4.2, U3.1
- new net: R10.2, U3.7, U5.7 (2A)
- new net: N10.1 (+), U5.11 (3Y)
- new net: N10.2 (-), U5.14 (4Y)
- new net: N9.1 (+), U5.3 (1Y)
- new net: N9.2 (-), U5.6 (2Y)
- new net M5V: C2.1, C3.1, J1.3 (VIN2), U1.3 (VOUT), U2.6, U2.8, U3.6, U3.8, U4.6, U4.8, U5.16 (VCC1)
- new net MOTOR_POWER: J1.2 (VOUT), U5.8 (VCC2)
- no-connect marks 24 -> 5
Other:
- note added: "Electrically Isolated"
- moved on the sheet: G1, H1, N1, N2

Commit message: Initial layout is complete.
Parts:
- removed N5, N6: HC_SR04_CONNECTOR, symbol HC_SR04_CONNECTOR
- U2, U3, U4: value OPTO_ISOLATOR -> LTV-826
- renumbered N9 to N5, N10 to N6
Connections:
- net D0: no longer N8.3 (TRIG)
- net D1: no longer N7.3 (TRIG)
- net D3: now also N8.3 (TRIG)
- net D9: now also N7.3 (TRIG)
- net M5V: now also C4.1
- net MGND: no longer C4.1
- net M2+: now reaches N6.1 (+), U5.11 (3Y)
- net M2-: now reaches N6.2 (-), U5.14 (4Y)
- net M1+: now reaches N5.1 (+), U5.3 (1Y)
- net M1-: now reaches N5.2 (-), U5.6 (2Y)
- no-connect marks 5 -> 9
Other:
- note added: "+"
- moved on the sheet: H1, N5, N6
Changed lines of the file:
@@
 L 3MM_HOLE H1
 U 1 1 53AA33AA
-P 4400 7000
-F 0 "H1" H 4350 7150 50  0000 C CNN
-F 1 "3MM_HOLE" H 4400 6850 50  0000 C CNN
-F 2 "" H 4400 7000 60  0000 C CNN
-F 3 "" H 4400 7000 60  0000 C CNN
-	1    4400 7000
+P 4400 5900
+F 0 "H1" H 4350 6050 50  0000 C CNN
+F 1 "3MM_HOLE" H 4400 5750 50  0000 C CNN
+F 2 "" H 4400 5900 60  0000 C CNN
+F 3 "" H 4400 5900 60  0000 C CNN
+	1    4400 5900
 	1    0    0    -1
 $EndComp
@@
 P 7000 2200
 F 0 "U2" H 6995 2510 60  0000 C CNN
-F 1 "OPTO_ISOLATOR" H 7000 1875 60  0000 C CNN
+F 1 "LTV-826" H 7000 1875 60  0000 C CNN
 F 2 "" H 7000 2200 60  0000 C CNN
 F 3 "" H 7000 2200 60  0000 C CNN
@@
 L GND #PWR01
 U 1 1 53B064D1
-P 4100 7500
-F 0 "#PWR01" H 4100 7500 30  0001 C CNN
-F 1 "GND" H 4100 7430 30  0001 C CNN
-F 2 "" H 4100 7500 60  0000 C CNN
-F 3 "" H 4100 7500 60  0000 C CNN
-	1    4100 7500
+P 4100 6100
+F 0 "#PWR01" H 4100 6100 30  0001 C CNN
+F 1 "GND" H 4100 6030 30  0001 C CNN
+F 2 "" H 4100 6100 60  0000 C CNN
+F 3 "" H 4100 6100 60  0000 C CNN
+	1    4100 6100
 	1    0    0    -1
 $EndComp
@@
 P 7000 3800
 F 0 "U3" H 6995 4110 60  0000 C CNN
-F 1 "OPTO_ISOLATOR" H 7000 3475 60  0000 C CNN
+F 1 "LTV-826" H 7000 3475 60  0000 C CNN
 F 2 "" H 7000 3800 60  0000 C CNN
 F 3 "" H 7000 3800 60  0000 C CNN
@@
 P 7000 5400
 F 0 "U4" H 6995 5710 60  0000 C CNN
-F 1 "OPTO_ISOLATOR" H 7000 5075 60  0000 C CNN
+F 1 "LTV-826" H 7000 5075 60  0000 C CNN
 F 2 "" H 7000 5400 60  0000 C CNN
 F 3 "" H 7000 5400 60  0000 C CNN
@@
 P 7000 1400
 F 0 "U2" H 6995 1710 60  0000 C CNN
-F 1 "OPTO_ISOLATOR" H 7000 1075 60  0000 C CNN
+F 1 "LTV-826" H 7000 1075 60  0000 C CNN
 F 2 "" H 7000 1400 60  0000 C CNN
 F 3 "" H 7000 1400 60  0000 C CNN
@@
 P 7000 3000
 F 0 "U3" H 6995 3310 60  0000 C CNN
-F 1 "OPTO_ISOLATOR" H 7000 2675 60  0000 C CNN
+F 1 "LTV-826" H 7000 2675 60  0000 C CNN
 F 2 "" H 7000 3000 60  0000 C CNN
 F 3 "" H 7000 3000 60  0000 C CNN
@@
 P 7000 4600
 F 0 "U4" H 6995 4910 60  0000 C CNN
-F 1 "OPTO_ISOLATOR" H 7000 4275 60  0000 C CNN
+F 1 "LTV-826" H 7000 4275 60  0000 C CNN
 F 2 "" H 7000 4600 60  0000 C CNN
 F 3 "" H 7000 4600 60  0000 C CNN
@@
 $EndComp
 $Comp
-L MOTOR_CONNECTOR N9
+L MOTOR_CONNECTOR N5
 U 1 1 53B16BD0
-P 10100 1950
-F 0 "N9" H 10100 2100 50  0000 C CNN
+P 10300 1950
+F 0 "N5" H 10300 2100 50  0000 C CNN
 F 1 "MOTOR_CONNECTOR" H 10100 1800 50  0000 C CNN
-F 2 "" H 10100 1950 60  0000 C CNN
-F 3 "" H 10100 1950 60  0000 C CNN
-	1    10100 1950
-	1    0    0    -1
-$EndComp
-$Comp
-L MOTOR_CONNECTOR N10
+F 2 "" H 10300 1950 60  0000 C CNN
+F 3 "" H 10300 1950 60  0000 C CNN
+	1    10300 1950
+	1    0    0    -1
+$EndComp
+$Comp
+L MOTOR_CONNECTOR N6
 U 1 1 53B16F6F
-P 10100 2450
-F 0 "N10" H 10100 2600 50  0000 C CNN
+P 10300 2450
+F 0 "N6" H 10300 2600 50  0000 C CNN
 F 1 "MOTOR_CONNECTOR" H 10100 2300 50  0000 C CNN
-F 2 "" H 10100 2450 60  0000 C CNN
-F 3 "" H 10100 2450 60  0000 C CNN
-	1    10100 2450
+F 2 "" H 10300 2450 60  0000 C CNN
+F 3 "" H 10300 2450 60  0000 C CNN
+	1    10300 2450
 	1    0    0    -1
 $EndComp
@@
 Text Notes 9600 6650 0    50   ~ 0
 Electrically Isolated
-$Comp
-L HC_SR04_CONNECTOR N5
-U 1 1 53B1AFF9
-P 4550 4650
-F 0 "N5" H 4550 4900 50  0000 C CNN
-F 1 "HC_SR04_CONNECTOR" H 4550 4400 50  0000 C CNN
-F 2 "" H 4550 4650 50  0000 C CNN
-F 3 "" H 4550 4650 50  0000 C CNN
-	1    4550 4650
-	1    0    0    -1
-$EndComp
 $Comp
 L ENCODER_CONNECTOR N3
@@
 	1    0    0    -1
 $EndComp
-$Comp
-L HC_SR04_CONNECTOR N6
-U 1 1 53B21AF3
-P 4550 5250
-F 0 "N6" H 4550 5500 50  0000 C CNN
-F 1 "HC_SR04_CONNECTOR" H 4550 5000 50  0000 C CNN
-F 2 "" H 4550 5250 50  0000 C CNN
-F 3 "" H 4550 5250 50  0000 C CNN
-	1    4550 5250
-	1    0    0    -1
-$EndComp
-$Comp
-L HC_SR04_CONNECTOR N7
-U 1 1 53B21F16
-P 4550 5850
-F 0 "N7" H 4550 6100 50  0000 C CNN
-F 1 "HC_SR04_CONNECTOR" H 4550 5600 50  0000 C CNN
-F 2 "" H 4550 5850 50  0000 C CNN
-F 3 "" H 4550 5850 50  0000 C CNN
-	1    4550 5850
-	1    0    0    -1
-$EndComp
-$Comp
-L HC_SR04_CONNECTOR N8
-U 1 1 53B21F66
-P 4550 6450
-F 0 "N8" H 4550 6700 50  0000 C CNN
-F 1 "HC_SR04_CONNECTOR" H 4550 6200 50  0000 C CNN
-F 2 "" H 4550 6450 50  0000 C CNN
-F 3 "" H 4550 6450 50  0000 C CNN
-	1    4550 6450
-	1    0    0    -1
-$EndComp
 NoConn ~ 2100 4600
 NoConn ~ 2100 4700
@@
 	2100 4500 1800 4500
 Wire Wire Line
-	1800 5400 2000 5400
-Wire Wire Line
-	2000 5400 2000 5500
-Wire Wire Line
-	4100 5500 1800 5500
-Wire Wire Line
-	1800 5800 2000 5800
-Wire Wire Line
-	2000 5800 2000 5900
-Wire Wire Line
-	2000 5900 1800 5900
-Connection ~ 2000 5500
+	1800 5400 4200 5400
+Wire Wire Line
+	2100 5500 1800 5500
+Wire Wire Line
+	1800 5800 2100 5800
+Wire Wire Line
+	2100 5800 2100 5900
+Wire Wire Line
+	2100 5900 1800 5900
 Wire Wire Line
 	1800 2600 5400 2600
@@
 	1800 2800 5200 2800
 Wire Wire Line
-	1800 2900 3500 2900
+	1800 2900 3400 2900
 Wire Wire Line
 	1800 3000 5100 3000
@@
 	1800 3400 3700 3400
 Wire Wire Line
-	1800 3500 3400 3500
+	1800 3500 3300 3500
 Wire Wire Line
 	1800 3600 3600 3600
 Wire Wire Line
-	1800 3700 3300 3700
-Wire Wire Line
-	1800 3800 3200 3800
+	1800 3700 2100 3700
+Wire Wire Line
+	1800 3800 2100 3800
 Wire Wire Line
 	1800 4600 2100 4600
@@
 	2100 4700 1800 4700
 Wire Wire Line
-	1800 4800 3100 4800
-Wire Wire Line
-	1800 4900 3100 4900
-Wire Wire Line
-	1800 5000 3000 5000
-Wire Wire Line
-	1800 5100 2900 5100
+	1800 4800 2100 4800
+Wire Wire Line
+	1800 4900 2100 4900
+Wire Wire Line
+	1800 5000 3100 5000
+Wire Wire Line
+	1800 5100 3100 5100
 Wire Wire Line
 	2100 5200 1800 5200
@@
 Wire Wire Line
 	2100 5600 1800 5600
-Wire Wire Line
-	1800 5700 4200 5700
 Wire Wire Line
 	3700 1400 3900 1400
@@
 	9700 2800 9700 2500
 Wire Wire Line
-	9700 2500 9800 2500
-Wire Wire Line
-	9800 2400 9600 2400
-Wire Wire Line
-	9800 2000 9600 2000
-Wire Wire Line
-	9800 1900 9700 1900
+	9700 2500 10000 2500
+Wire Wire Line
+	10000 2400 9600 2400
+Wire Wire Line
+	10000 2000 9600 2000
+Wire Wire Line
+	10000 1900 9700 1900
 Wire Wire Line
 	9700 1900 9700 1600
@@
 	8600 3100 8400 3100
 Connection ~ 8400 3100
-Wire Wire Line
-	5700 800  8200 800
 Connection ~ 8400 3000
 Wire Wire Line
@@
 	6000 4000 5900 4000
 Wire Wire Line
-	5200 5600 6500 5600
-Wire Wire Line
 	6400 1600 6400 5600
 Wire Wire Line
@@
 	4200 4200 4100 4200
 Wire Wire Line
-	4100 3600 4100 7500
-Wire Wire Line
 	4100 3600 4200 3600
 Wire Wire Line
 	4200 3300 4000 3300
 Wire Wire Line
-	4000 3300 4000 6300
+	4000 3300 4000 5700
 Wire Wire Line
 	4000 3900 4200 3900
@@
 Wire Wire Line
 	3600 4100 3600 3600
-Wire Wire Line
-	4200 4600 3500 4600
-Wire Wire Line
-	3500 4600 3500 2900
-Wire Wire Line
-	4200 5200 3400 5200
-Wire Wire Line
-	3400 5200 3400 3500
-Wire Wire Line
-	4200 5800 3300 5800
-Wire Wire Line
-	3300 5800 3300 3700
-Wire Wire Line
-	4200 6400 3200 6400
-Wire Wire Line
-	3200 6400 3200 3800
-Wire Wire Line
-	4000 6300 4200 6300
 Connection ~ 4000 3900
-Connection ~ 4000 5700
-Wire Wire Line
-	4200 5100 4000 5100
-Connection ~ 4000 5100
-Wire Wire Line
-	4200 4500 4000 4500
-Connection ~ 4000 4500
-Wire Wire Line
-	4100 6600 4200 6600
 Connection ~ 4100 4200
-Wire Wire Line
-	4200 4800 4100 4800
-Connection ~ 4100 4800
-Wire Wire Line
-	4200 5400 4100 5400
-Connection ~ 4100 5400
-Wire Wire Line
-	4200 6000 4100 6000
-Connection ~ 4100 6000
-Wire Wire Line
-	4200 6500 2900 6500
-Wire Wire Line
-	2900 6500 2900 5100
-Wire Wire Line
-	3000 5900 4200 5900
-Wire Wire Line
-	3000 5000 3000 5900
-Wire Wire Line
-	4200 5300 3100 5300
-Wire Wire Line
-	3100 5300 3100 4900
-Wire Wire Line
-	4200 4700 3100 4700
-Wire Wire Line
-	3100 4700 3100 4800
-Wire Wire Line
-	4100 7000 4200 7000
-Connection ~ 4100 6600
-Connection ~ 4100 7000
-Connection ~ 4100 5500
 Wire Wire Line
 	8400 1500 7950 1500
@@
 	8200 1500 8200 1400
 Connection ~ 8200 1500
-Wire Wire Line
-	8200 800  8200 1000
-Connection ~ 7950 800
-Wire Wire Line
-	5200 5600 5200 7300
-Wire Wire Line
-	5200 7300 4100 7300
-Connection ~ 4100 7300
 Connection ~ 6400 5600
 Wire Wire Line
@@
 Wire Wire Line
 	7800 5900 7800 1600
+Wire Wire Line
+	4200 5900 4100 5900
+NoConn ~ 2100 4800
+NoConn ~ 2100 4900
+Wire Wire Line
+	4000 5700 1800 5700
+Text Label 9750 1900 0    50   ~ 0
+M1+
+Text Label 9750 2000 0    50   ~ 0
+M1-
+Text Label 9750 2400 0    50   ~ 0
+M2+
+Text Label 9750 2500 0    50   ~ 0
+M2-
+Wire Wire Line
+	7950 800  5700 800
+Wire Wire Line
+	8200 1000 8200 700
+Connection ~ 8200 700
+$Comp
+L HC_SR04_CONNECTOR N7
+U 1 1 53B4C06A
+P 4550 4650
+F 0 "N7" H 4550 4900 50  0000 C CNN
+F 1 "HC_SR04_CONNECTOR" H 4550 4400 50  0000 C CNN
+F 2 "" H 4550 4650 50  0000 C CNN
+F 3 "" H 4550 4650 50  0000 C CNN
+	1    4550 4650
+	1    0    0    -1
+$EndComp
+$Comp
+L HC_SR04_CONNECTOR N8
+U 1 1 53B4C21C
+P 4550 5250
+F 0 "N8" H 4550 5500 50  0000 C CNN
+F 1 "HC_SR04_CONNECTOR" H 4550 5000 50  0000 C CNN
+F 2 "" H 4550 5250 50  0000 C CNN
+F 3 "" H 4550 5250 50  0000 C CNN
+	1    4550 5250
+	1    0    0    -1
+$EndComp
+Connection ~ 4100 5600
+Wire Wire Line
+	4200 4500 4000 4500
+Connection ~ 4000 4500
+Wire Wire Line
+	4200 5100 4000 5100
+Connection ~ 4000 5100
+Connection ~ 4100 5400
+Wire Wire Line
+	4200 4800 4100 4800
+Connection ~ 4100 4800
+Wire Wire Line
+	4200 4600 3400 4600
+Wire Wire Line
+	3400 4600 3400 2900
+Wire Wire Line
+	4200 5200 3300 5200
+Wire Wire Line
+	3300 5200 3300 3500
+Wire Wire Line
+	4200 5300 3100 5300
+Wire Wire Line
+	3100 5300 3100 5100
+Wire Wire Line
+	3100 5000 3100 4700
+Wire Wire Line
+	3100 4700 4200 4700
+Connection ~ 4100 5900
+Wire Wire Line
+	4100 3600 4100 6100
+NoConn ~ 2100 3700
+NoConn ~ 2100 3800
+Connection ~ 2100 5400
+Wire Wire Line
+	4100 5600 6500 5600
+Wire Wire Line
+	2100 5500 2100 5400
+Text Notes 3600 1650 0    50   ~ 0
++
+Text Notes 5300 1650 0    50   ~ 0
++
 $EndSCHEMATC
